File: hardware/mouse.kicad_sch (KiCad schematic)
At the start: 52 parts, among them J1 USB_B_Micro, J2 JSTPH, SW1 SW_SPST, SW2 SW_SPST, SW3 SW_SPST, SW4 SW_SPST, SW5 SW_SPST, SW6 SW_SPST, U1 ATSAMD21G18A-A, U2 SPX3819M5-L-3-3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

Commit message: finished the first version of the schematic
Parts:
- removed J1: USB_B_Micro, symbol Connector:USB_B_Micro
- added J3: USB_C_Receptacle_USB2.0_14P, symbol Connector:USB_C_Receptacle_USB2.0_14P
- added R14, R15: 5.1kΩ, symbol Device:R_US
- added R16, R17: 220Ω, symbol Device:R_US
- added SW7: RotaryEncoder, symbol Device:RotaryEncoder
- added SW7: SW_SPST, symbol Switch:SW_SPST
- renumbered SW3 to SW2, SW4 to SW3, SW5 to SW4, SW6 to SW5, SW2 to SW6
Connections:
- net LEDBLUEOUT is gone; now on net GND: D1.1 (KB)
- net LEDGREENOUT is gone; now on net GND: D1.3 (KG)
- net +3.3V: now also SW7.C
- net D+: now also J3.A6 (D+), J3.B6 (D+)
- net D-: now also J3.A7 (D-), J3.B7 (D-)
- net GND: now also J3.A1 (GND), J3.A12 (GND), J3.B1 (GND), J3.B12 (GND), R14.2, R15.1, R16.1, R17.2, SW7.1 (A)
- net LEDBLUEIN: now also U1.25 (PA16), R16.2
- net LEDGREENIN: now also R17.1
- net MISO: now also U1.21 (PA12)
- net MOSI: now also U1.19 (PB10)
- net MOTION: now also U1.15 (PA10)
- net NCS: now also U1.16 (PA11)
- net NRESET: now also SW7.2 (B)
- net SCLK: now also U1.20 (PB11)
- net Switch1: now also U1.30 (PA21)
- net Switch2: now also U1.29 (PA20)
- net Switch3: now also U1.28 (PA19)
- net Switch4: now also U1.27 (PA18)
- net Switch5: now also U1.26 (PA17)
- net VBUS: now also J3.A4 (VBUS), J3.A9 (VBUS), J3.B4 (VBUS), J3.B9 (VBUS)
- net RECCW: now reaches U1.13 (PA08)
- net RECCW: now also SW7.B
- net RECW: now reaches U1.14 (PA09)
- net RECW: now also SW7.A
- new net USBCC1: J3.A5 (CC1), R14.1
- new net USBCC2: J3.B5 (CC2), R15.2
Other:
- note added: "Rotary Encoder"
- note added: "Switches"
- moved on the sheet: SW6
