File: hardware/mouse/mouse.kicad_pcb (KiCad board)
At the start: 4 copper layers, 44 x 68 mm, 88 parts, among them J2 JSTPH, J3 USB_C_Receptacle_USB2.0_14P, SW1 SW_SPST, SW2 SW_SPST, SW3 SW_SPST, SW4 SW_SPST, SW5 SW_SPST, SW6 SW_SPST, SW7 SW_SPST, SW8 RotaryEncoder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

Commit message: idr what changed
Parts:
- removed C40, C9: 10uF, Capacitor_SMD:C_0805_2012Metric_Pad1.18x1.45mm_HandSolder
- removed D1, D2, D4, D6: MBR1020VL, Diode_SMD:D_SOD-123F
- C1: value 4.7uF -> 4.7μF
- C10, C12, C15, C16, C18, C3, C41, C43, C6, C8: value 10uF -> 10μF
- C11, C17, C42: value 1uF -> 1μF
- C30, C32: value 1.0μF -> 1μF
- J3: footprint Connector_USB:USB_C_Receptacle_Amphenol_12401548E4-2A -> custom:AMPHENOL_12401598E4_2A
- moved J3 4.39 mm to (126.4, 83.2)
Routing:
- net Net-(J3-SHIELD): track 25.5 -> 1.36 mm
- net Net-(D1-K): track 20.4 -> 0.00 mm, vias 3 -> 0
- net +BATT: track 110.3 -> 96.4 mm, vias 8 -> 6
- net Net-(J3-CC1): track 25.5 -> 13.5 mm, vias 2 -> 3
- net Net-(D3-K): track 69.9 -> 58.1 mm
- net Net-(D2-K): track 7.57 -> 0.00 mm, vias 3 -> 0
- net GND: track 161.4 -> 155.5 mm, vias 10 -> 9
- net VBUS: track 120.2 -> 115.6 mm, vias 7 -> 8
- net D-: track 36.7 -> 40.4 mm, vias 2 -> 3
- net D+: track 36.8 -> 37.7 mm, vias 2 -> 3
