File: hardware/mouse/mouse.kicad_sch (KiCad schematic)
At the start: 63 parts, among them J2 JSTPH, J3 USB_C_Receptacle_USB2.0_14P, SW1 SW_SPST, SW2 SW_SPST, SW3 SW_SPST, SW4 SW_SPST, SW5 SW_SPST, SW6 SW_SPST, SW7 SW_SPST, SW8 RotaryEncoder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

Commit message: added bom to README
Parts:
- C1: value 4.7uF -> 4.7μF
- C10, C12, C15, C16, C18, C3, C41, C43, C6, C8: value 10uF -> 10μF
- C11, C17, C42: value 1uF -> 1μF
Changed lines of the file:
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@@
 			)
 		)
-		(property "Value" "1uF"
+		(property "Value" "1μF"
 			(at 76.2 115.5699 0)
 			(effects
@@
 			)
 		)
-		(property "Value" "1uF"
+		(property "Value" "1μF"
 			(at 76.2 152.3999 0)
 			(effects
@@
 			)
 		)
-		(property "Value" "10uF"
+		(property "Value" "10μF"
 			(at 121.92 184.1499 0)
 			(effects
@@
 			)
 		)
-		(property "Value" "10uF"
+		(property "Value" "10μF"
 			(at 64.77 187.9599 0)
 			(effects
@@
 			)
 		)
-		(property "Value" "1uF"
+		(property "Value" "1μF"
 			(at 76.2 187.9599 0)
 			(effects
@@
 			)
 		)
-		(property "Value" "10uF"
+		(property "Value" "10μF"
 			(at 238.76 121.9199 0)
 			(effects
@@
 			)
 		)
-		(property "Value" "10uF"
+		(property "Value" "10μF"
 			(at 64.77 115.5699 0)
 			(effects
@@
 			)
 		)
-		(property "Value" "10uF"
+		(property "Value" "10μF"
 			(at 34.29 147.3199 0)
 			(effects
@@
 			)
 		)
-		(property "Value" "10uF"
+		(property "Value" "10μF"
 			(at 134.62 184.1499 0)
 			(effects
@@
 			)
 		)
-		(property "Value" "10uF"
+		(property "Value" "10μF"
 			(at 240.03 38.0999 0)
 			(effects
@@
 			)
 		)
-		(property "Value" "10uF"
+		(property "Value" "10μF"
 			(at 204.47 152.3999 0)
 			(effects
@@
 			)
 		)
-		(property "Value" "4.7uF"
+		(property "Value" "4.7μF"
 			(at 195.58 129.5399 0)
 			(effects
@@
 			)
 		)
-		(property "Value" "10uF"
+		(property "Value" "10μF"
 			(at 64.77 152.3999 0)
 			(effects
@@
 			)
 		)
-		(property "Value" "10uF"
+		(property "Value" "10μF"
 			(at 109.22 184.1499 0)
 			(effects

Commit message: idr what changed
Parts:
- J3: footprint Connector_USB:USB_C_Receptacle_Amphenol_12401548E4-2A -> custom:AMPHENOL_12401598E4_2A
Changed lines of the file:
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@@
 			)
 		)
-		(property "Footprint" "Connector_USB:USB_C_Receptacle_Amphenol_12401548E4-2A"
+		(property "Footprint" "custom:AMPHENOL_12401598E4_2A"
 			(at 162.56 38.1 0)
 			(effects
