File: hardware/mouse/rfradio.kicad_sch (KiCad schematic)
At the start: 19 parts, among them U5 nRF52840

Commit message: idr what changed
Parts:
- C30, C32: value 1.0μF -> 1μF
Changed lines of the file:
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@@
 			)
 		)
-		(property "Value" "1.0μF"
+		(property "Value" "1μF"
 			(at 18.288 116.586 0)
 			(effects
@@
 			)
 		)
-		(property "Value" "1.0μF"
+		(property "Value" "1μF"
 			(at 222.25 148.59 90)
 			(effects
